Commit message: added color to the sign

File: lettering_config/urdf/sign_macro.xacro (robot description, xacro)
@@ -7,4 +7,7 @@
         <mesh filename="package://lettering_config/meshes/signs/${prefix}.stl"/>
       </geometry>
+      <material>
+        <color rgba="0 0 .8 1"/>
+      </material>
     </visual>
     <collision>
@@ -12,4 +15,7 @@
         <mesh filename="package://lettering_config/meshes/collision/${prefix}.stl" />
       </geometry>
+      <material>
+        <color rgba="1 1 1 1"/>
+      </material>
     </collision>
   </link>
@@ -23,4 +29,7 @@
         <mesh filename="package://lettering_config/meshes/letters/${prefix}.stl" />
       </geometry>
+      <material>
+        <color rgba="1 1 1 1"/>
+      </material>
     </visual>
   </link>

Commit message: trivial change

File: lettering_config/urdf/sign_macro.xacro (robot description, xacro)
@@ -20,5 +20,5 @@
     </collision>
   </link>
-  <joint name="${prefix}_joint_1" type="fixed">
+  <joint name="${prefix}_joint" type="fixed">
     <parent link="${prefix}_sign"/>
     <child link="${prefix}_letters"/>

Commit message: corrected stl to STL

File: lettering_config/urdf/sign_macro.xacro (robot description, xacro)
@@ -5,5 +5,5 @@
     <visual>
       <geometry>
-        <mesh filename="package://lettering_config/meshes/signs/${prefix}.stl"/>
+        <mesh filename="package://lettering_config/meshes/signs/${prefix}.STL"/>
       </geometry>
       <material>
@@ -13,5 +13,5 @@
     <collision>
       <geometry>
-        <mesh filename="package://lettering_config/meshes/collision/${prefix}.stl" />
+        <mesh filename="package://lettering_config/meshes/collision/${prefix}.STL" />
       </geometry>
       <material>
@@ -27,5 +27,5 @@
     <visual>
       <geometry>
-        <mesh filename="package://lettering_config/meshes/letters/${prefix}.stl" />
+        <mesh filename="package://lettering_config/meshes/letters/${prefix}.STL" />
       </geometry>
       <material>

Commit message: added name attribute to material element

File: lettering_config/urdf/sign_macro.xacro (robot description, xacro)
@@ -7,5 +7,5 @@
         <mesh filename="package://lettering_config/meshes/signs/${prefix}.STL"/>
       </geometry>
-      <material>
+      <material name="blue">
         <color rgba="0 0 .8 1"/>
       </material>
@@ -15,5 +15,5 @@
         <mesh filename="package://lettering_config/meshes/collision/${prefix}.STL" />
       </geometry>
-      <material>
+      <material name="white">
         <color rgba="1 1 1 1"/>
       </material>
@@ -29,7 +29,5 @@
         <mesh filename="package://lettering_config/meshes/letters/${prefix}.STL" />
       </geometry>
-      <material>
-        <color rgba="1 1 1 1"/>
-      </material>
+      <material name="white"/>
     </visual>
   </link>

Commit message: fixed the colors

File: lettering_config/urdf/sign_macro.xacro (robot description, xacro)
@@ -7,6 +7,6 @@
         <mesh filename="package://lettering_config/meshes/signs/${prefix}.STL"/>
       </geometry>
-      <material name="blue">
-        <color rgba="0 0 .8 1"/>
+      <material name="white">
+        <color rgba="1 1 1 1"/>
       </material>
     </visual>
@@ -15,7 +15,5 @@
         <mesh filename="package://lettering_config/meshes/collision/${prefix}.STL" />
       </geometry>
-      <material name="white">
-        <color rgba="1 1 1 1"/>
-      </material>
+      <material name="white"/>
     </collision>
   </link>
@@ -29,5 +27,7 @@
         <mesh filename="package://lettering_config/meshes/letters/${prefix}.STL" />
       </geometry>
-      <material name="white"/>
+      <material name="blue">
+        <color rgba="0 0 .8 1"/>
+      </material>
     </visual>
   </link>
